File: atividade2/atividade2.sch (KiCad schematic (older format))
At the start: 13 parts, among them J1 USB_B_Micro, J2 Conn_02x10_Odd_Even, U1 STM32F030, U2 LD1117S33TR_SOT223

Commit message: finished
Parts:
- removed C1: 10nF, Capacitor_SMD:C_0805_2012Metric_Pad1.15x1.40mm_HandSolder, symbol Device:C
- removed C2: 1uF, Capacitor_SMD:C_0805_2012Metric_Pad1.15x1.40mm_HandSolder, symbol Device:C
- removed C3: 0.1uF, Capacitor_SMD:C_0805_2012Metric_Pad1.15x1.40mm_HandSolder, symbol Device:C
- removed C4: 100nF, Capacitor_SMD:C_0805_2012Metric_Pad1.15x1.40mm_HandSolder, symbol Device:C
- removed C5: 4.7uF, Capacitor_SMD:C_0805_2012Metric_Pad1.15x1.40mm_HandSolder, symbol Device:C
- removed D1, D2: LED, LED_SMD:LED_0805_2012Metric_Pad1.15x1.40mm_HandSolder, symbol Device:LED
- removed D3: Status, LED_SMD:LED_0805_2012Metric_Pad1.15x1.40mm_HandSolder, symbol Device:LED
- removed J1: USB_B_Micro, Connector_USB:USB_Micro-B_Molex-105017-0001, symbol Connector:USB_B_Micro
- removed J2: Conn_02x10_Odd_Even, Connector_PinHeader_2.00mm:PinHeader_2x10_P2.00mm_Vertical, symbol Connector_Generic:Conn_02x10_Odd_Even
- removed R1: 39, Resistor_SMD:R_0805_2012Metric_Pad1.15x1.40mm_HandSolder, symbol Device:R_US
- removed U1: STM32F030, Package_SO:TSSOP-20_4.4x6.5mm_P0.65mm, symbol atividade2:STM32F030
- removed U2: LD1117S33TR_SOT223, Package_TO_SOT_SMD:SOT-223-3_TabPin2, symbol Regulator_Linear:LD1117S33TR_SOT223
Connections:
- net labels removed: +3.3V, +5V, GND, NRST, SPI1_MISO, SPI1_MOSI, SPI1_NSS, SPI1_SCK, SWCLK, SWDIO, USART1_RX, USART1_TX
- wire segments 45 -> 0
- no-connect marks 12 -> 0
